File: Combined_PCB/inputs_filtering.kicad_sch (KiCad schematic)
At the start: 20 parts, among them J1 Conn_01x08_Pin, J2 Conn_01x08_Pin, J4 Conn_01x02_Pin, J6 Conn_01x08_Socket, J7 Conn_01x08_Socket, U10 TPD4E1B06DRLR, U11 TPD4E1B06DRLR, U12 TPD4E1B06DRLR, U8 TPD4E1B06DRLR, U9 TPD4E1B06DRLR

Commit message: Semi-finalized PCB Layout final
Parts:
- removed J6, J7: Conn_01x08_Socket, symbol Connector:Conn_01x08_Socket
- added J6, J7: Conn_01x01_Pin, symbol Connector:Conn_01x01_Pin
Connections:
- new net DAISY_IN: J6.1 (Pin_1)
- new net DGND: J7.1 (Pin_1)

Commit message: Schematic and footprints complete
Parts:
- C1: renamed from C9; footprint W3A45C102K4T2A:CAPCAF50P200X125X85-8 -> W3A45C102K4T2A:CAPCAV_W3A45C102KAT2A-8
- C2: renamed from C11; footprint W3A45C102K4T2A:CAPCAF50P200X125X85-8 -> W3A45C102K4T2A:CAPCAV_W3A45C102KAT2A-8
- C3: renamed from C24; footprint W3A45C102K4T2A:CAPCAF50P200X125X85-8 -> W3A45C102K4T2A:CAPCAV_W3A45C102KAT2A-8
- C4: renamed from C25; footprint W3A45C102K4T2A:CAPCAF50P200X125X85-8 -> W3A45C102K4T2A:CAPCAV_W3A45C102KAT2A-8
- C5: renamed from C26; footprint W3A45C102K4T2A:CAPCAF50P200X125X85-8 -> W3A45C102K4T2A:CAPCAV_W3A45C102KAT2A-8
- J1: footprint Connector_PinHeader_2.54mm:PinHeader_1x08_P2.54mm_Vertical -> Connector_PinHeader_2.54mm:PinHeader_1x08_P2.54mm_Horizontal
- J2: renamed from J4; footprint (none) -> Connector_PinHeader_2.54mm:PinHeader_1x02_P2.54mm_Horizontal
- J3: renamed from J2; footprint Connector_PinHeader_2.54mm:PinHeader_1x08_P2.54mm_Vertical -> Connector_PinHeader_2.54mm:PinHeader_1x08_P2.54mm_Horizontal
- J4: renamed from J6; footprint (none) -> TestPoint:TestPoint_Pad_D2.5mm
- J5: renamed from J7; footprint (none) -> TestPoint:TestPoint_Pad_D2.5mm
- U1: renamed from U8; footprint TPD4E1B06:DRL6_TEX -> DRL6:DRL6_TEX
- U2: renamed from U9; footprint TPD4E1B06:DRL6_TEX -> DRL6:DRL6_TEX
- U3: renamed from U10; footprint TPD4E1B06:DRL6_TEX -> DRL6:DRL6_TEX
- U4: renamed from U11; footprint TPD4E1B06:DRL6_TEX -> DRL6:DRL6_TEX
- U5: renamed from U12; footprint TPD4E1B06:DRL6_TEX -> DRL6:DRL6_TEX
- renumbered RN6 to RN1, RN7 to RN2, RN8 to RN3, RN9 to RN4, RN10 to RN5
Connections:
- no-connect marks 7 -> 3

Commit message: ADS1299 final pcb layout done (hopefully)
Parts:
- J1, J3: footprint Connector_PinHeader_2.54mm:PinHeader_1x08_P2.54mm_Horizontal -> Connector_JST:JST_XH_S8B-XH-A_1x08_P2.50mm_Horizontal
- J2: footprint Connector_PinHeader_2.54mm:PinHeader_1x02_P2.54mm_Horizontal -> Connector_JST:JST_XH_S2B-XH-A_1x02_P2.50mm_Horizontal
Connections:
- net 1N: now also J3.2 (Pin_2), RN4.7 (R2.2), U4.6 (IO4); no longer J3.8 (Pin_8), RN4.8 (R1.2), U4.4 (IO3)
- net 1P: now also J3.1 (Pin_1), RN4.8 (R1.2), U4.4 (IO3); no longer J3.7 (Pin_7), RN4.7 (R2.2), U4.6 (IO4)
- net 2N: now also J3.4 (Pin_4), RN4.5 (R4.2), U4.3 (IO2); no longer J3.6 (Pin_6), RN4.6 (R3.2), U4.1 (IO1)
- net 2P: now also J3.3 (Pin_3), RN4.6 (R3.2), U4.1 (IO1); no longer J3.5 (Pin_5), RN4.5 (R4.2), U4.3 (IO2)
- net 3N: now also J3.6 (Pin_6), RN3.7 (R2.2), U3.6 (IO4); no longer J3.4 (Pin_4), RN3.8 (R1.2), U3.4 (IO3)
- net 3P: now also J3.5 (Pin_5), RN3.8 (R1.2), U3.4 (IO3); no longer J3.3 (Pin_3), RN3.7 (R2.2), U3.6 (IO4)
- net 4N: now also J3.8 (Pin_8), RN3.5 (R4.2), U3.3 (IO2); no longer J3.2 (Pin_2), RN3.6 (R3.2), U3.1 (IO1)
- net 4P: now also J3.7 (Pin_7), RN3.6 (R3.2), U3.1 (IO1); no longer J3.1 (Pin_1), RN3.5 (R4.2), U3.3 (IO2)
- net 5N: now also J1.2 (Pin_2), RN2.7 (R2.2), U2.6 (IO4); no longer J1.8 (Pin_8), RN2.8 (R1.2), U2.4 (IO3)
- net 5P: now also J1.1 (Pin_1), RN2.8 (R1.2), U2.4 (IO3); no longer J1.7 (Pin_7), RN2.7 (R2.2), U2.6 (IO4)
- net 6N: now also J1.4 (Pin_4), RN2.5 (R4.2), U2.3 (IO2); no longer J1.6 (Pin_6), RN2.6 (R3.2), U2.1 (IO1)
- net 6P: now also J1.3 (Pin_3), RN2.6 (R3.2), U2.1 (IO1); no longer J1.5 (Pin_5), RN2.5 (R4.2), U2.3 (IO2)
- net 7N: now also J1.6 (Pin_6), RN1.7 (R2.2), U1.6 (IO4); no longer J1.4 (Pin_4), RN1.8 (R1.2), U1.4 (IO3)
- net 7P: now also J1.5 (Pin_5), RN1.8 (R1.2), U1.4 (IO3); no longer J1.3 (Pin_3), RN1.7 (R2.2), U1.6 (IO4)
- net 8N: now also J1.8 (Pin_8), RN1.5 (R4.2), U1.3 (IO2); no longer J1.2 (Pin_2), RN1.6 (R3.2), U1.1 (IO1)
- net 8P: now also J1.7 (Pin_7), RN1.6 (R3.2), U1.1 (IO1); no longer J1.1 (Pin_1), RN1.5 (R4.2), U1.3 (IO2)
- net BIAS: now also J2.2 (Pin_2), U5.3 (IO2); no longer J2.1 (Pin_1), U5.1 (IO1)
- net BIASINV: now also J2.1 (Pin_1), U5.1 (IO1); no longer J2.2 (Pin_2), U5.3 (IO2)
- net IN1N: now also C4.7, RN4.2 (R2.1); no longer C4.8, RN4.1 (R1.1)
- net IN1P: now also C4.8, RN4.1 (R1.1); no longer C4.7, RN4.2 (R2.1)
- net IN2N: now also C4.5, RN4.4 (R4.1); no longer C4.6, RN4.3 (R3.1)
- net IN2P: now also C4.6, RN4.3 (R3.1); no longer C4.5, RN4.4 (R4.1)
- net IN3N: now also C3.7, RN3.2 (R2.1); no longer C3.8, RN3.1 (R1.1)
- net IN3P: now also C3.8, RN3.1 (R1.1); no longer C3.7, RN3.2 (R2.1)
- net IN4N: now also C3.5, RN3.4 (R4.1); no longer C3.6, RN3.3 (R3.1)
- net IN4P: now also C3.6, RN3.3 (R3.1); no longer C3.5, RN3.4 (R4.1)
- net IN5N: now also C2.7, RN2.2 (R2.1); no longer C2.8, RN2.1 (R1.1)
- net IN5P: now also C2.8, RN2.1 (R1.1); no longer C2.7, RN2.2 (R2.1)
- net IN6N: now also C2.5, RN2.4 (R4.1); no longer C2.6, RN2.3 (R3.1)
- net IN6P: now also C2.6, RN2.3 (R3.1); no longer C2.5, RN2.4 (R4.1)
- net IN7N: now also C1.7, RN1.2 (R2.1); no longer C1.8, RN1.1 (R1.1)
- net IN7P: now also C1.8, RN1.1 (R1.1); no longer C1.7, RN1.2 (R2.1)
- net IN8N: now also C1.5, RN1.4 (R4.1); no longer C1.6, RN1.3 (R3.1)
- net IN8P: now also C1.6, RN1.3 (R3.1); no longer C1.5, RN1.4 (R4.1)
