File: Combined_PCB/Combined_PCB.kicad_pcb (KiCad board)
At the start: 4 copper layers, 35.6 x 74.4 mm, 43 parts, among them J1 Conn_01x08_Pin, J2 Conn_01x02_Pin, J3 Conn_01x08_Pin, J6 Conn_01x18_Pin, J7 Conn_01x18_Pin, U1 TPD4E1B06DRLR, U2 TPD4E1B06DRLR, U3 TPD4E1B06DRLR, U4 TPD4E1B06DRLR, U5 TPD4E1B06DRLR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

Commit message: Add CS
Parts:
- renumbered DI to J4, GND to J5
Connections:
- J6 pad 11: /ADS1299 & Microcontroller/START -> /ADS1299 & Microcontroller/CS
- J6 pad 12: unconnected-(J6-Pin_12-Pad12) -> /ADS1299 & Microcontroller/START
- U6 pad 39: AGND -> /ADS1299 & Microcontroller/CS
Routing:
- net /ADS1299 & Microcontroller/CS: track 0.00 -> 17.6 mm, vias 0 -> 1
- net AGND: track 44.1 -> 42.3 mm
- net /ADS1299 & Microcontroller/START: track 17.4 -> 15.7 mm
- net /ADS1299 & Microcontroller/MOSI: track 23.1 -> 23.8 mm
Other:
- board size 35.6 x 74.4 mm -> 35.6 x 77.5 mm

Commit message: Final PCB Render Done
Connections:
- U6 pad 17: AGND -> /ADS1299 & Microcontroller/SRB1
- U6 pad 18: AGND -> /ADS1299 & Microcontroller/SRB2
Changed lines of the file:
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@@
 	(net 92 "unconnected-(J7-Pin_18-Pad18)")
 	(net 93 "unconnected-(J7-Pin_6-Pad6)")
+	(net 94 "/ADS1299 & Microcontroller/SRB1")
+	(net 95 "/ADS1299 & Microcontroller/SRB2")
 	(footprint "DRL6:DRL6_TEX"
 		(layer "F.Cu")
@@
 			(pintype "bidirectional")
 		)
+		(model "${KICAD8_3DMODEL_DIR}/Package_TO_SOT_SMD.3dshapes/SOT-563.step"
+			(offset
+				(xyz 0 0 0)
+			)
+			(scale
+				(xyz 1 1 1)
+			)
+			(rotate
+				(xyz 0 0 0)
+			)
+		)
 	)
 	(footprint "Capacitor_SMD:C_0805_2012Metric"
@@
 				(font
 					(size 0.48 0.48)
-					(thickness 0.15)
+					(thickness 0.12)
 				)
 			)
@@
 				(font
 					(size 0.48 0.48)
-					(thickness 0.15)
+					(thickness 0.12)
 				)
 			)
@@
 			(solder_mask_margin 0.102)
 		)
+		(model "${KIPRJMOD}/ProjectLibraries/W3A45C102K4T2A/W3A45C102K4T2A.step"
+			(offset
+				(xyz 0 0 0)
+			)
+			(scale
+				(xyz 1 1 1)
+			)
+			(rotate
+				(xyz -90 0 0)
+			)
+		)
 	)
 	(footprint "Capacitor_SMD:C_0805_2012Metric"
@@
 			(pintype "bidirectional")
 		)
+		(model "${KICAD8_3DMODEL_DIR}/Package_TO_SOT_SMD.3dshapes/SOT-563.step"
+			(offset
+				(xyz 0 0 0)
+			)
+			(scale
+				(xyz 1 1 1)
+			)
+			(rotate
+				(xyz 0 0 0)
+			)
+		)
 	)
 	(footprint "DRL6:DRL6_TEX"
@@
 			(pintype "bidirectional+no_connect")
 		)
+		(model "${KICAD8_3DMODEL_DIR}/Package_TO_SOT_SMD.3dshapes/SOT-563.step"
+			(offset
+				(xyz 0 0 0)
+			)
+			(scale
+				(xyz 1 1 1)
+			)
+			(rotate
+				(xyz 0 0 0)
+			)
+		)
 	)
 	(footprint "Capacitor_SMD:C_0805_2012Metric"
@@
 				(font
 					(size 0.48 0.48)
-					(thickness 0.15)
+					(thickness 0.12)
 				)
 			)
@@
 				(font
 					(size 0.48 0.48)
-					(thickness 0.15)
+					(thickness 0.12)
 				)
 			)
@@
 			(solder_mask_margin 0.102)
 		)
+		(model "${KIPRJMOD}/ProjectLibraries/W3A45C102K4T2A/W3A45C102K4T2A.step"
+			(offset
+				(xyz 0 0 0)
+			)
+			(scale
+				(xyz 1 1 1)
+			)
+			(rotate
+				(xyz -90 0 0)
+			)
+		)
 	)
 	(footprint "Resistor_SMD:R_0805_2012Metric"
@@
 				(font
 					(size 0.48 0.48)
-					(thickness 0.15)
+					(thickness 0.12)
 				)
 			)
@@
 				(font
 					(size 0.48 0.48)
-					(thickness 0.15)
+					(thickness 0.12)
 				)
 			)
@@
 			(solder_mask_margin 0.102)
 		)
+		(model "${KIPRJMOD}/ProjectLibraries/W3A45C102K4T2A/W3A45C102K4T2A.step"
+			(offset
+				(xyz 0 0 0)
+			)
+			(scale
+				(xyz 1 1 1)
+			)
+			(rotate
+				(xyz -90 0 0)
+			)
+		)
 	)
 	(footprint "Capacitor_SMD:C_0805_2012Metric"
@@
 				(font
 					(size 0.48 0.48)
-					(thickness 0.15)
+					(thickness 0.12)
 				)
 			)
@@
 				(font
 					(size 0.48 0.48)
-					(thickness 0.15)
+					(thickness 0.12)
 				)
 			)
@@
 			(solder_mask_margin 0.102)
 		)
+		(model "${KIPRJMOD}/ProjectLibraries/W3A45C102K4T2A/W3A45C102K4T2A.step"
+			(offset
+				(xyz 0 0 0)
+			)
+			(scale
+				(xyz 1 1 1)
+			)
+			(rotate
+				(xyz -90 0 0)
+			)
+		)
 	)
 	(footprint "Capacitor_SMD:C_0805_2012Metric"
@@
 		(at 119.38 66.04 -90)
 		(property "Reference" "U6"
-			(at 0 0 180)
+			(at 0 0 360)
 			(layer "F.SilkS")
 			(effects
@@
 		)
 		(property "Value" "ADS1299IPAG"
-			(at 20.555 -10.845 -90)
+			(at 20.555 -10.845 90)
 			(layer "F.Fab")
 			(effects
@@
 			(layers "F.Cu" "F.Paste" "F.Mask")
 			(roundrect_rratio 0.125)
-			(net 2 "AGND")
+			(net 94 "/ADS1299 & Microcontroller/SRB1")
 			(pinfunction "SRB1")
 			(pintype "bidirectional")
@@
 			(layers "F.Cu" "F.Paste" "F.Mask")
 			(roundrect_rratio 0.125)
-			(net 2 "AGND")
+			(net 95 "/ADS1299 & Microcontroller/SRB2")
 			(pinfunction "SRB2")
 			(pintype "bidirectional")
@@
 			(solder_mask_margin 0.102)
 		)
+		(model "${KIPRJMOD}/ProjectLibraries/ADS1299/ADS1299IPAG.step"
+			(offset
+				(xyz 0 0 0)
+			)
+			(scale
+				(xyz 1 1 1)
+			)
+			(rotate
+				(xyz -90 0 0)
+			)
+		)
 	)
 	(footprint "Resistor_SMD:R_Array_Concave_4x0603"
@@
 				(font
 					(size 0.48 0.48)
-					(thickness 0.15)
+					(thickness 0.12)
 				)
 			)
@@
 				(font
 					(size 0.48 0.48)
-					(thickness 0.15)
+					(thickness 0.12)
 				)
 			)
@@
 			(solder_mask_margin 0.102)
 		)
+		(model "${KIPRJMOD}/ProjectLibraries/W3A45C102K4T2A/W3A45C102K4T2A.step"
+			(offset
+				(xyz 0 0 0)
+			)
+			(scale
+				(xyz 1 1 1)
+			)
+			(rotate
+				(xyz -90 0 0)
+			)
+		)
 	)
 	(footprint "Resistor_SMD:R_Array_Concave_4x0603"
@@
 			(pintype "bidirectional")
 		)
+		(model "${KICAD8_3DMODEL_DIR}/Package_TO_SOT_SMD.3dshapes/SOT-563.step"
+			(offset
+				(xyz 0 0 0)
+			)
+			(scale
+				(xyz 1 1 1)
+			)
+			(rotate
+				(xyz 0 0 0)
+			)
+		)
 	)
 	(footprint "Capacitor_SMD:C_0805_2012Metric"
@@
 			(pintype "input")
 		)
+		(model "${KIPRJMOD}/ProjectLibraries/MCP1640/MCP1640.step"
+			(offset
+				(xyz 0 0 0)
+			)
+			(scale
+				(xyz 1 1 1)
+			)
+			(rotate
+				(xyz 0 0 0)
+			)
+		)
 	)
 	(footprint "DRL6:DRL6_TEX"
@@
 			(pintype "bidirectional")
 		)
+		(model "${KICAD8_3DMODEL_DIR}/Package_TO_SOT_SMD.3dshapes/SOT-563.step"
+			(offset
+				(xyz 0 0 0)
+			)
+			(scale
+				(xyz 1 1 1)
+			)
+			(rotate
+				(xyz 0 0 0)
+			)
+		)
 	)
